Commit message: Update the robot descriptions
- Format the XMLs based on mujoco_menagerie
- Format the floats in XMLs to 8 decimals
- Increase the shoulder pitch limits to -270 to 270

File: toddlerbot/descriptions/toddlerbot_2xc/toddlerbot_2xc.urdf (robot description, URDF)
Before this commit: robot toddlerbot_2xc, 91 links, 90 joints
Joints:
- joint left_ankle_pitch: origin xyz=-7.16755e-18 -1.03457e-16 -0.11 rpy=0.0 0.0 0.0 -> xyz=0.0 0.0 -0.11 rpy=0.0 0.0 0.0
- joint left_ankle_roll: origin xyz=-0.023 0.019 1.74061e-14 rpy=0.0 0.0 0.0 -> xyz=-0.023 0.019 0.0 rpy=0.0 0.0 0.0
- joint left_elbow_roll: origin xyz=-0.019 9.63118e-18 -0.061 rpy=0.0 0.0 0.0 -> xyz=-0.019 0.0 -0.061 rpy=0.0 0.0 0.0
- joint left_elbow_yaw_driven: origin xyz=0.019 3.58087e-10 -0.025 rpy=0.0 0.0 0.0 -> xyz=0.019 0.0 -0.025 rpy=0.0 0.0 0.0
- joint left_hip_pitch: limit lower=-2.356194490192225 upper=1.832595714594166 effort=100 velocity=100 -> lower=-2.356194490192345 upper=1.8325957145940461 effort=100 velocity=100
- joint left_hip_yaw_drive: origin xyz=-0.0192 -0.0002 1.13154e-14 rpy=0.0 0.0 0.0 -> xyz=-0.0192 -0.0002 0.0 rpy=0.0 0.0 0.0
- joint left_hip_yaw_driven: origin xyz=-0.019 5.2261e-16 -0.033 rpy=0.0 0.0 0.0 -> xyz=-0.019 0.0 -0.033 rpy=0.0 0.0 0.0
- joint left_knee: origin xyz=-5.41634e-16 -0.019 -0.0445 rpy=0.0 0.0 0.0 -> xyz=0.0 -0.019 -0.0445 rpy=0.0 0.0 0.0
- joint left_shoulder_pitch: limit lower=-3.1415926535897913 upper=3.141592653589795 effort=100 velocity=100 -> lower=-4.712388980384688 upper=4.7123889803846915 effort=100 velocity=100
- joint left_shoulder_roll: origin xyz=-0.019 0.027 5.964920000000001e-18 rpy=0.0 0.0 0.0 -> xyz=-0.019 0.027 0.0 rpy=0.0 0.0 0.0
- joint left_shoulder_yaw_driven: origin xyz=0.019 3.58104e-10 -0.025 rpy=0.0 0.0 0.0 -> xyz=0.019 0.0 -0.025 rpy=0.0 0.0 0.0
- joint left_wrist_pitch_drive: origin xyz=1.52463e-10 -0.003 0.024 rpy=0.0 0.0 0.0 -> xyz=0.0 -0.003 0.024 rpy=0.0 0.0 0.0
- joint left_wrist_pitch_driven: origin xyz=4.76147e-17 0.022 -0.061 rpy=0.0 0.0 0.0 -> xyz=0.0 0.022 -0.061 rpy=0.0 0.0 0.0
- joint left_wrist_roll: origin xyz=-0.019 -0.022 -3.58074e-10 rpy=0.0 0.0 0.0 -> xyz=-0.019 -0.022 0.0 rpy=0.0 0.0 0.0
- joint neck_pitch: limit lower=-0.6108652381980295 upper=1.3962634015954494 effort=100 velocity=100 -> lower=-0.6108652381980767 upper=1.3962634015954023 effort=100 velocity=100; origin xyz=9.24195e-17 0.004 0.015 rpy=0.0 0.0 0.0 -> xyz=0.0 0.004 0.015 rpy=0.0 0.0 0.0
- joint neck_yaw_drive: origin xyz=-0.0215079 1.21496e-14 0.119 rpy=0.0 0.0 0.0 -> xyz=-0.0215079 0.0 0.119 rpy=0.0 0.0 0.0
- joint neck_yaw_driven: origin xyz=-0.00050787 -1.1277e-19 0.124 rpy=0.0 0.0 0.0 -> xyz=-0.00050787 0.0 0.124 rpy=0.0 0.0 0.0
- joint right_ankle_pitch: origin xyz=-7.14345e-18 -1.9508e-16 -0.11 rpy=0.0 0.0 0.0 -> xyz=0.0 0.0 -0.11 rpy=0.0 0.0 0.0
- joint right_ankle_roll: origin xyz=-0.023 -0.019 4.5011e-15 rpy=0.0 0.0 0.0 -> xyz=-0.023 -0.019 0.0 rpy=0.0 0.0 0.0
- joint right_elbow_roll: origin xyz=0.019 3.1225e-17 -0.061 rpy=0.0 0.0 0.0 -> xyz=0.019 0.0 -0.061 rpy=0.0 0.0 0.0
- joint right_elbow_yaw_driven: origin xyz=-0.019 -3.58088e-10 -0.025 rpy=0.0 0.0 0.0 -> xyz=-0.019 0.0 -0.025 rpy=0.0 0.0 0.0
- joint right_hip_pitch: limit lower=-1.8325957145940204 upper=2.3561944901923706 effort=100 velocity=100 -> lower=-1.8325957145940186 upper=2.3561944901923724 effort=100 velocity=100
- joint right_hip_yaw_drive: origin xyz=-0.0192 0.0002 1.12316e-14 rpy=0.0 0.0 0.0 -> xyz=-0.0192 0.0002 0.0 rpy=0.0 0.0 0.0
- joint right_hip_yaw_driven: origin xyz=0.019 -5.8123e-16 -0.033 rpy=0.0 0.0 0.0 -> xyz=0.019 0.0 -0.033 rpy=0.0 0.0 0.0
- joint right_knee: origin xyz=5.05409e-16 0.019 -0.0445 rpy=0.0 0.0 0.0 -> xyz=0.0 0.019 -0.0445 rpy=0.0 0.0 0.0
- joint right_shoulder_pitch: limit lower=-3.14159265358977 upper=3.141592653589816 effort=100 velocity=100 -> lower=-4.71238898038469 upper=4.71238898038469 effort=100 velocity=100
- joint right_shoulder_roll: origin xyz=0.019 -0.027 1.03253e-17 rpy=0.0 0.0 0.0 -> xyz=0.019 -0.027 0.0 rpy=0.0 0.0 0.0
- joint right_shoulder_yaw_driven: origin xyz=-0.019 -3.58104e-10 -0.025 rpy=0.0 0.0 0.0 -> xyz=-0.019 0.0 -0.025 rpy=0.0 0.0 0.0
- joint right_wrist_pitch_drive: origin xyz=-1.52463e-10 0.003 0.024 rpy=0.0 0.0 0.0 -> xyz=0.0 0.003 0.024 rpy=0.0 0.0 0.0
- joint right_wrist_pitch_driven: origin xyz=-8.69443e-17 -0.022 -0.061 rpy=0.0 0.0 0.0 -> xyz=0.0 -0.022 -0.061 rpy=0.0 0.0 0.0
- joint right_wrist_roll: origin xyz=0.019 0.022 -3.58075e-10 rpy=0.0 0.0 0.0 -> xyz=0.019 0.022 0.0 rpy=0.0 0.0 0.0
- joint waist_act_1: origin xyz=-0.01275 -1.71841e-16 -0.0196 rpy=0.0 0.0 0.0 -> xyz=-0.01275 0.0 -0.0196 rpy=0.0 0.0 0.0
- joint waist_act_2: origin xyz=-0.03275 1.40567e-16 -0.0196 rpy=0.0 0.0 0.0 -> xyz=-0.03275 0.0 -0.0196 rpy=0.0 0.0 0.0
- joint waist_roll: limit lower=-0.5235987755983015 upper=0.5235987755982962 effort=100 velocity=100 -> lower=-0.5235987755983006 upper=0.523598775598297 effort=100 velocity=100; origin xyz=0.0230079 2.89995e-16 -0.014 rpy=0.0 0.0 0.0 -> xyz=0.0230079 0.0 -0.014 rpy=0.0 0.0 0.0
- joint waist_yaw: limit lower=-1.570796326794878 upper=1.5707963267949152 effort=100 velocity=100 -> lower=-1.5707963267948895 upper=1.5707963267949037 effort=100 velocity=100; origin xyz=-0.0165079 -1.92151e-17 -0.00248651 rpy=0.0 0.0 0.0 -> xyz=-0.0165079 0.0 -0.00248651 rpy=0.0 0.0 0.0

File: toddlerbot/descriptions/toddlerbot_2xc_gripper/toddlerbot_2xc_gripper.urdf (robot description, URDF)
Before this commit: robot toddlerbot_2xc_gripper, 103 links, 102 joints
Joints:
- joint left_ankle_pitch: origin xyz=-7.16755e-18 -1.03457e-16 -0.11 rpy=0.0 0.0 0.0 -> xyz=0.0 0.0 -0.11 rpy=0.0 0.0 0.0
- joint left_ankle_roll: origin xyz=-0.023 0.019 1.74061e-14 rpy=0.0 0.0 0.0 -> xyz=-0.023 0.019 0.0 rpy=0.0 0.0 0.0
- joint left_elbow_roll: origin xyz=-0.019 -6.66967e-17 -0.061 rpy=0.0 0.0 0.0 -> xyz=-0.019 0.0 -0.061 rpy=0.0 0.0 0.0
- joint left_elbow_yaw_driven: origin xyz=0.019 3.58086e-10 -0.025 rpy=0.0 0.0 0.0 -> xyz=0.019 0.0 -0.025 rpy=0.0 0.0 0.0
- joint left_hip_pitch: limit lower=-2.356194490192225 upper=1.832595714594166 effort=100 velocity=100 -> lower=-2.356194490192345 upper=1.8325957145940461 effort=100 velocity=100
- joint left_hip_yaw_drive: origin xyz=-0.0192 -0.0002 1.13154e-14 rpy=0.0 0.0 0.0 -> xyz=-0.0192 -0.0002 0.0 rpy=0.0 0.0 0.0
- joint left_hip_yaw_driven: origin xyz=-0.019 5.2261e-16 -0.033 rpy=0.0 0.0 0.0 -> xyz=-0.019 0.0 -0.033 rpy=0.0 0.0 0.0
- joint left_knee: origin xyz=-5.41634e-16 -0.019 -0.0445 rpy=0.0 0.0 0.0 -> xyz=0.0 -0.019 -0.0445 rpy=0.0 0.0 0.0
- joint left_shoulder_pitch: limit lower=-3.1415926535897913 upper=3.141592653589795 effort=100 velocity=100 -> lower=-4.712388980384688 upper=4.7123889803846915 effort=100 velocity=100
- joint left_shoulder_roll: origin xyz=-0.019 0.027 -1.67365e-15 rpy=0.0 0.0 0.0 -> xyz=-0.019 0.027 0.0 rpy=0.0 0.0 0.0
- joint left_shoulder_yaw_driven: origin xyz=0.019 3.58104e-10 -0.025 rpy=0.0 0.0 0.0 -> xyz=0.019 0.0 -0.025 rpy=0.0 0.0 0.0
- joint left_wrist_pitch_drive: origin xyz=1.52465e-10 -0.003 0.024 rpy=0.0 0.0 0.0 -> xyz=0.0 -0.003 0.024 rpy=0.0 0.0 0.0
- joint left_wrist_pitch_driven: origin xyz=2.52308e-17 0.022 -0.061 rpy=0.0 0.0 0.0 -> xyz=0.0 0.022 -0.061 rpy=0.0 0.0 0.0
- joint left_wrist_roll: origin xyz=-0.019 -0.022 -3.58073e-10 rpy=0.0 0.0 0.0 -> xyz=-0.019 -0.022 0.0 rpy=0.0 0.0 0.0
- joint neck_pitch: limit lower=-0.6108652381980295 upper=1.3962634015954494 effort=100 velocity=100 -> lower=-0.6108652381980779 upper=1.396263401595401 effort=100 velocity=100; origin xyz=9.24195e-17 0.004 0.015 rpy=0.0 0.0 0.0 -> xyz=0.0 0.004 0.015 rpy=0.0 0.0 0.0
- joint neck_yaw_drive: origin xyz=-0.0215079 1.21496e-14 0.119 rpy=0.0 0.0 0.0 -> xyz=-0.0215079 0.0 0.119 rpy=0.0 0.0 0.0
- joint neck_yaw_driven: origin xyz=-0.00050787 -1.1277e-19 0.124 rpy=0.0 0.0 0.0 -> xyz=-0.00050787 0.0 0.124 rpy=0.0 0.0 0.0
- joint right_ankle_pitch: origin xyz=-7.14345e-18 -1.9508e-16 -0.11 rpy=0.0 0.0 0.0 -> xyz=0.0 0.0 -0.11 rpy=0.0 0.0 0.0
- joint right_ankle_roll: origin xyz=-0.023 -0.019 4.5011e-15 rpy=0.0 0.0 0.0 -> xyz=-0.023 -0.019 0.0 rpy=0.0 0.0 0.0
- joint right_elbow_roll: origin xyz=0.019 -6.245e-17 -0.061 rpy=0.0 0.0 0.0 -> xyz=0.019 0.0 -0.061 rpy=0.0 0.0 0.0
- joint right_elbow_yaw_driven: origin xyz=-0.019 -3.58087e-10 -0.025 rpy=0.0 0.0 0.0 -> xyz=-0.019 0.0 -0.025 rpy=0.0 0.0 0.0
- joint right_hip_pitch: limit lower=-1.8325957145940204 upper=2.3561944901923706 effort=100 velocity=100 -> lower=-1.8325957145940186 upper=2.3561944901923724 effort=100 velocity=100
- joint right_hip_yaw_drive: origin xyz=-0.0192 0.0002 1.12316e-14 rpy=0.0 0.0 0.0 -> xyz=-0.0192 0.0002 0.0 rpy=0.0 0.0 0.0
- joint right_hip_yaw_driven: origin xyz=0.019 -5.8123e-16 -0.033 rpy=0.0 0.0 0.0 -> xyz=0.019 0.0 -0.033 rpy=0.0 0.0 0.0
- joint right_knee: origin xyz=5.05409e-16 0.019 -0.0445 rpy=0.0 0.0 0.0 -> xyz=0.0 0.019 -0.0445 rpy=0.0 0.0 0.0
- joint right_shoulder_pitch: limit lower=-3.14159265358977 upper=3.141592653589816 effort=100 velocity=100 -> lower=-4.71238898038469 upper=4.71238898038469 effort=100 velocity=100
- joint right_shoulder_roll: origin xyz=0.019 -0.027 -1.42914e-16 rpy=0.0 0.0 0.0 -> xyz=0.019 -0.027 0.0 rpy=0.0 0.0 0.0
- joint right_shoulder_yaw_driven: origin xyz=-0.019 -3.58104e-10 -0.025 rpy=0.0 0.0 0.0 -> xyz=-0.019 0.0 -0.025 rpy=0.0 0.0 0.0
- joint right_wrist_pitch_drive: origin xyz=-1.52465e-10 0.003 0.024 rpy=0.0 0.0 0.0 -> xyz=0.0 0.003 0.024 rpy=0.0 0.0 0.0
- joint right_wrist_pitch_driven: origin xyz=1.47538e-15 -0.022 -0.061 rpy=0.0 0.0 0.0 -> xyz=0.0 -0.022 -0.061 rpy=0.0 0.0 0.0
- joint right_wrist_roll: origin xyz=0.019 0.022 -3.58073e-10 rpy=0.0 0.0 0.0 -> xyz=0.019 0.022 0.0 rpy=0.0 0.0 0.0
- joint waist_act_1: origin xyz=-0.01275 -1.71841e-16 -0.0196 rpy=0.0 0.0 0.0 -> xyz=-0.01275 0.0 -0.0196 rpy=0.0 0.0 0.0
- joint waist_act_2: origin xyz=-0.03275 1.40567e-16 -0.0196 rpy=0.0 0.0 0.0 -> xyz=-0.03275 0.0 -0.0196 rpy=0.0 0.0 0.0
- joint waist_roll: limit lower=-0.5235987755983015 upper=0.5235987755982962 effort=100 velocity=100 -> lower=-0.5235987755983006 upper=0.523598775598297 effort=100 velocity=100; origin xyz=0.0230079 2.89995e-16 -0.014 rpy=0.0 0.0 0.0 -> xyz=0.0230079 0.0 -0.014 rpy=0.0 0.0 0.0
- joint waist_yaw: limit lower=-1.570796326794878 upper=1.5707963267949152 effort=100 velocity=100 -> lower=-1.570796326794894 upper=1.5707963267948992 effort=100 velocity=100; origin xyz=-0.0165079 -1.92151e-17 -0.00248651 rpy=0.0 0.0 0.0 -> xyz=-0.0165079 0.0 -0.00248651 rpy=0.0 0.0 0.0

File: toddlerbot/descriptions/toddlerbot_2xm/toddlerbot_2xm.urdf (robot description, URDF)
Before this commit: robot toddlerbot_2xm, 91 links, 90 joints
Links:
- link right_hip_pitch_link: geometry collision box size=0.0857375 0.0424 0.0465 type=box; visual mesh filename=assets/right_hip_pitch_link_visual.stl scale=1.0 1.0 1.0
Joints:
- joint left_ankle_pitch: origin xyz=-7.16755e-18 -4.83405e-17 -0.11 rpy=0.0 0.0 0.0 -> xyz=0.0 0.0 -0.11 rpy=0.0 0.0 0.0
- joint left_ankle_roll: origin xyz=-0.023 0.019 1.74256e-14 rpy=0.0 0.0 0.0 -> xyz=-0.023 0.019 0.0 rpy=0.0 0.0 0.0
- joint left_elbow_roll: origin xyz=-0.019 9.63118e-18 -0.061 rpy=0.0 0.0 0.0 -> xyz=-0.019 0.0 -0.061 rpy=0.0 0.0 0.0
- joint left_elbow_yaw_driven: origin xyz=0.019 3.58087e-10 -0.025 rpy=0.0 0.0 0.0 -> xyz=0.019 0.0 -0.025 rpy=0.0 0.0 0.0
- joint left_hip_pitch: limit lower=-2.356194490192225 upper=0.7853981633975682 effort=100 velocity=100 -> lower=-2.356194490192345 upper=0.7853981633974483 effort=100 velocity=100
- joint left_hip_yaw_drive: origin xyz=-0.0192 -0.0002 1.12946e-14 rpy=0.0 0.0 0.0 -> xyz=-0.0192 -0.0002 0.0 rpy=0.0 0.0 0.0
- joint left_hip_yaw_driven: origin xyz=0.023 -6.96693e-16 -0.033 rpy=0.0 0.0 0.0 -> xyz=0.023 0.0 -0.033 rpy=0.0 0.0 0.0
- joint left_knee: origin xyz=-4.78197e-16 -0.019 -0.0445 rpy=0.0 0.0 0.0 -> xyz=0.0 -0.019 -0.0445 rpy=0.0 0.0 0.0
- joint left_shoulder_pitch: limit lower=-3.1415926535897913 upper=3.141592653589795 effort=100 velocity=100 -> lower=-4.712388980384688 upper=4.7123889803846915 effort=100 velocity=100
- joint left_shoulder_roll: origin xyz=-0.019 0.027 5.964920000000001e-18 rpy=0.0 0.0 0.0 -> xyz=-0.019 0.027 0.0 rpy=0.0 0.0 0.0
- joint left_shoulder_yaw_driven: origin xyz=0.019 3.58104e-10 -0.025 rpy=0.0 0.0 0.0 -> xyz=0.019 0.0 -0.025 rpy=0.0 0.0 0.0
- joint left_wrist_pitch_drive: origin xyz=1.52463e-10 -0.003 0.024 rpy=0.0 0.0 0.0 -> xyz=0.0 -0.003 0.024 rpy=0.0 0.0 0.0
- joint left_wrist_pitch_driven: origin xyz=4.76147e-17 0.022 -0.061 rpy=0.0 0.0 0.0 -> xyz=0.0 0.022 -0.061 rpy=0.0 0.0 0.0
- joint left_wrist_roll: origin xyz=-0.019 -0.022 -3.58074e-10 rpy=0.0 0.0 0.0 -> xyz=-0.019 -0.022 0.0 rpy=0.0 0.0 0.0
- joint neck_pitch: limit lower=-0.6108652381980295 upper=1.3962634015954494 effort=100 velocity=100 -> lower=-0.6108652381980779 upper=1.396263401595401 effort=100 velocity=100; origin xyz=9.24195e-17 0.004 0.015 rpy=0.0 0.0 0.0 -> xyz=0.0 0.004 0.015 rpy=0.0 0.0 0.0
- joint neck_yaw_drive: origin xyz=-0.0215079 1.21496e-14 0.119 rpy=0.0 0.0 0.0 -> xyz=-0.0215079 0.0 0.119 rpy=0.0 0.0 0.0
- joint neck_yaw_driven: origin xyz=-0.00050787 -1.1277e-19 0.124 rpy=0.0 0.0 0.0 -> xyz=-0.00050787 0.0 0.124 rpy=0.0 0.0 0.0
- joint right_ankle_pitch: origin xyz=-1.14853e-17 -2.25611e-16 -0.11 rpy=0.0 0.0 0.0 -> xyz=0.0 0.0 -0.11 rpy=0.0 0.0 0.0
- joint right_ankle_roll: origin xyz=-0.023 -0.019 1.78974e-14 rpy=0.0 0.0 0.0 -> xyz=-0.023 -0.019 0.0 rpy=0.0 0.0 0.0
- joint right_elbow_roll: origin xyz=0.019 3.1225e-17 -0.061 rpy=0.0 0.0 0.0 -> xyz=0.019 0.0 -0.061 rpy=0.0 0.0 0.0
- joint right_elbow_yaw_driven: origin xyz=-0.019 -3.58088e-10 -0.025 rpy=0.0 0.0 0.0 -> xyz=-0.019 0.0 -0.025 rpy=0.0 0.0 0.0
- joint right_hip_pitch: limit lower=-0.7853981633974225 upper=2.3561944901923706 effort=100 velocity=100 -> lower=-0.7853981633974207 upper=2.3561944901923724 effort=100 velocity=100
- joint right_hip_yaw_drive: origin xyz=-0.0192 0.0002 1.12316e-14 rpy=0.0 0.0 0.0 -> xyz=-0.0192 0.0002 0.0 rpy=0.0 0.0 0.0
- joint right_hip_yaw_driven: origin xyz=0.023 -6.96693e-16 -0.033 rpy=0.0 0.0 0.0 -> xyz=0.023 0.0 -0.033 rpy=0.0 0.0 0.0
- joint right_knee: origin xyz=5.00205e-16 0.019 -0.0445 rpy=0.0 0.0 0.0 -> xyz=0.0 0.019 -0.0445 rpy=0.0 0.0 0.0
- joint right_shoulder_pitch: limit lower=-3.14159265358977 upper=3.141592653589816 effort=100 velocity=100 -> lower=-4.71238898038469 upper=4.71238898038469 effort=100 velocity=100
- joint right_shoulder_roll: origin xyz=0.019 -0.027 1.03253e-17 rpy=0.0 0.0 0.0 -> xyz=0.019 -0.027 0.0 rpy=0.0 0.0 0.0
- joint right_shoulder_yaw_driven: origin xyz=-0.019 -3.58104e-10 -0.025 rpy=0.0 0.0 0.0 -> xyz=-0.019 0.0 -0.025 rpy=0.0 0.0 0.0
- joint right_wrist_pitch_drive: origin xyz=-1.52463e-10 0.003 0.024 rpy=0.0 0.0 0.0 -> xyz=0.0 0.003 0.024 rpy=0.0 0.0 0.0
- joint right_wrist_pitch_driven: origin xyz=-8.69443e-17 -0.022 -0.061 rpy=0.0 0.0 0.0 -> xyz=0.0 -0.022 -0.061 rpy=0.0 0.0 0.0
- joint right_wrist_roll: origin xyz=0.019 0.022 -3.58075e-10 rpy=0.0 0.0 0.0 -> xyz=0.019 0.022 0.0 rpy=0.0 0.0 0.0
- joint waist_act_1: origin xyz=-0.01275 -1.71841e-16 -0.0196 rpy=0.0 0.0 0.0 -> xyz=-0.01275 0.0 -0.0196 rpy=0.0 0.0 0.0
- joint waist_act_2: origin xyz=-0.03275 1.40567e-16 -0.0196 rpy=0.0 0.0 0.0 -> xyz=-0.03275 0.0 -0.0196 rpy=0.0 0.0 0.0
- joint waist_roll: limit lower=-0.5235987755983015 upper=0.5235987755982962 effort=100 velocity=100 -> lower=-0.5235987755983006 upper=0.523598775598297 effort=100 velocity=100; origin xyz=0.0230079 2.89995e-16 -0.014 rpy=0.0 0.0 0.0 -> xyz=0.0230079 0.0 -0.014 rpy=0.0 0.0 0.0
- joint waist_yaw: limit lower=-1.570796326794878 upper=1.5707963267949152 effort=100 velocity=100 -> lower=-1.570796326794894 upper=1.5707963267948992 effort=100 velocity=100; origin xyz=-0.0165079 -1.92151e-17 -0.00248651 rpy=0.0 0.0 0.0 -> xyz=-0.0165079 0.0 -0.00248651 rpy=0.0 0.0 0.0

File: toddlerbot/descriptions/toddlerbot_2xm_gripper/toddlerbot_2xm_gripper.urdf (robot description, URDF)
Before this commit: robot toddlerbot_2xm_gripper, 103 links, 102 joints
Links:
- link right_hip_pitch_link: geometry collision box size=0.0857375 0.0424 0.0465 type=box; visual mesh filename=assets/right_hip_pitch_link_visual.stl scale=1.0 1.0 1.0
Joints:
- joint left_ankle_pitch: origin xyz=-7.16755e-18 -4.83405e-17 -0.11 rpy=0.0 0.0 0.0 -> xyz=0.0 0.0 -0.11 rpy=0.0 0.0 0.0
- joint left_ankle_roll: origin xyz=-0.023 0.019 1.74256e-14 rpy=0.0 0.0 0.0 -> xyz=-0.023 0.019 0.0 rpy=0.0 0.0 0.0
- joint left_elbow_roll: origin xyz=-0.019 -6.66967e-17 -0.061 rpy=0.0 0.0 0.0 -> xyz=-0.019 0.0 -0.061 rpy=0.0 0.0 0.0
- joint left_elbow_yaw_driven: origin xyz=0.019 3.58086e-10 -0.025 rpy=0.0 0.0 0.0 -> xyz=0.019 0.0 -0.025 rpy=0.0 0.0 0.0
- joint left_hip_pitch: limit lower=-2.356194490192225 upper=0.7853981633975682 effort=100 velocity=100 -> lower=-2.356194490192345 upper=0.7853981633974483 effort=100 velocity=100
- joint left_hip_yaw_drive: origin xyz=-0.0192 -0.0002 1.12946e-14 rpy=0.0 0.0 0.0 -> xyz=-0.0192 -0.0002 0.0 rpy=0.0 0.0 0.0
- joint left_hip_yaw_driven: origin xyz=0.023 -6.96693e-16 -0.033 rpy=0.0 0.0 0.0 -> xyz=0.023 0.0 -0.033 rpy=0.0 0.0 0.0
- joint left_knee: origin xyz=-4.78197e-16 -0.019 -0.0445 rpy=0.0 0.0 0.0 -> xyz=0.0 -0.019 -0.0445 rpy=0.0 0.0 0.0
- joint left_shoulder_pitch: limit lower=-3.1415926535897913 upper=3.141592653589795 effort=100 velocity=100 -> lower=-4.712388980384688 upper=4.7123889803846915 effort=100 velocity=100
- joint left_shoulder_roll: origin xyz=-0.019 0.027 -1.67365e-15 rpy=0.0 0.0 0.0 -> xyz=-0.019 0.027 0.0 rpy=0.0 0.0 0.0
- joint left_shoulder_yaw_driven: origin xyz=0.019 3.58104e-10 -0.025 rpy=0.0 0.0 0.0 -> xyz=0.019 0.0 -0.025 rpy=0.0 0.0 0.0
- joint left_wrist_pitch_drive: origin xyz=1.52465e-10 -0.003 0.024 rpy=0.0 0.0 0.0 -> xyz=0.0 -0.003 0.024 rpy=0.0 0.0 0.0
- joint left_wrist_pitch_driven: origin xyz=2.52308e-17 0.022 -0.061 rpy=0.0 0.0 0.0 -> xyz=0.0 0.022 -0.061 rpy=0.0 0.0 0.0
- joint left_wrist_roll: origin xyz=-0.019 -0.022 -3.58073e-10 rpy=0.0 0.0 0.0 -> xyz=-0.019 -0.022 0.0 rpy=0.0 0.0 0.0
- joint neck_pitch: limit lower=-0.6108652381980295 upper=1.3962634015954494 effort=100 velocity=100 -> lower=-0.6108652381980779 upper=1.396263401595401 effort=100 velocity=100; origin xyz=9.24195e-17 0.004 0.015 rpy=0.0 0.0 0.0 -> xyz=0.0 0.004 0.015 rpy=0.0 0.0 0.0
- joint neck_yaw_drive: origin xyz=-0.0215079 1.21496e-14 0.119 rpy=0.0 0.0 0.0 -> xyz=-0.0215079 0.0 0.119 rpy=0.0 0.0 0.0
- joint neck_yaw_driven: origin xyz=-0.00050787 -1.1277e-19 0.124 rpy=0.0 0.0 0.0 -> xyz=-0.00050787 0.0 0.124 rpy=0.0 0.0 0.0
- joint right_ankle_pitch: origin xyz=-1.14853e-17 -2.25611e-16 -0.11 rpy=0.0 0.0 0.0 -> xyz=0.0 0.0 -0.11 rpy=0.0 0.0 0.0
- joint right_ankle_roll: origin xyz=-0.023 -0.019 1.78974e-14 rpy=0.0 0.0 0.0 -> xyz=-0.023 -0.019 0.0 rpy=0.0 0.0 0.0
- joint right_elbow_roll: origin xyz=0.019 -6.245e-17 -0.061 rpy=0.0 0.0 0.0 -> xyz=0.019 0.0 -0.061 rpy=0.0 0.0 0.0
- joint right_elbow_yaw_driven: origin xyz=-0.019 -3.58087e-10 -0.025 rpy=0.0 0.0 0.0 -> xyz=-0.019 0.0 -0.025 rpy=0.0 0.0 0.0
- joint right_hip_pitch: limit lower=-0.7853981633974225 upper=2.3561944901923706 effort=100 velocity=100 -> lower=-0.7853981633974207 upper=2.3561944901923724 effort=100 velocity=100
- joint right_hip_yaw_drive: origin xyz=-0.0192 0.0002 1.12316e-14 rpy=0.0 0.0 0.0 -> xyz=-0.0192 0.0002 0.0 rpy=0.0 0.0 0.0
- joint right_hip_yaw_driven: origin xyz=0.023 -6.96693e-16 -0.033 rpy=0.0 0.0 0.0 -> xyz=0.023 0.0 -0.033 rpy=0.0 0.0 0.0
- joint right_knee: origin xyz=5.00205e-16 0.019 -0.0445 rpy=0.0 0.0 0.0 -> xyz=0.0 0.019 -0.0445 rpy=0.0 0.0 0.0
- joint right_shoulder_pitch: limit lower=-3.14159265358977 upper=3.141592653589816 effort=100 velocity=100 -> lower=-4.71238898038469 upper=4.71238898038469 effort=100 velocity=100
- joint right_shoulder_roll: origin xyz=0.019 -0.027 -1.42914e-16 rpy=0.0 0.0 0.0 -> xyz=0.019 -0.027 0.0 rpy=0.0 0.0 0.0
- joint right_shoulder_yaw_driven: origin xyz=-0.019 -3.58104e-10 -0.025 rpy=0.0 0.0 0.0 -> xyz=-0.019 0.0 -0.025 rpy=0.0 0.0 0.0
- joint right_wrist_pitch_drive: origin xyz=-1.52465e-10 0.003 0.024 rpy=0.0 0.0 0.0 -> xyz=0.0 0.003 0.024 rpy=0.0 0.0 0.0
- joint right_wrist_pitch_driven: origin xyz=1.47538e-15 -0.022 -0.061 rpy=0.0 0.0 0.0 -> xyz=0.0 -0.022 -0.061 rpy=0.0 0.0 0.0
- joint right_wrist_roll: origin xyz=0.019 0.022 -3.58073e-10 rpy=0.0 0.0 0.0 -> xyz=0.019 0.022 0.0 rpy=0.0 0.0 0.0
- joint waist_act_1: origin xyz=-0.01275 -1.71841e-16 -0.0196 rpy=0.0 0.0 0.0 -> xyz=-0.01275 0.0 -0.0196 rpy=0.0 0.0 0.0
- joint waist_act_2: origin xyz=-0.03275 1.40567e-16 -0.0196 rpy=0.0 0.0 0.0 -> xyz=-0.03275 0.0 -0.0196 rpy=0.0 0.0 0.0
- joint waist_roll: limit lower=-0.5235987755983015 upper=0.5235987755982962 effort=100 velocity=100 -> lower=-0.5235987755983006 upper=0.523598775598297 effort=100 velocity=100; origin xyz=0.0230079 2.89995e-16 -0.014 rpy=0.0 0.0 0.0 -> xyz=0.0230079 0.0 -0.014 rpy=0.0 0.0 0.0
- joint waist_yaw: limit lower=-1.570796326794878 upper=1.5707963267949152 effort=100 velocity=100 -> lower=-1.570796326794894 upper=1.5707963267948992 effort=100 velocity=100; origin xyz=-0.0165079 -1.92151e-17 -0.00248651 rpy=0.0 0.0 0.0 -> xyz=-0.0165079 0.0 -0.00248651 rpy=0.0 0.0 0.0
